File: BackpackPCB/ProtogenBackpackPCB.kicad_sch (KiCad schematic)
At the start: 22 parts, among them J1 Pololu D24V10F3, J2 Pololu D36V28F5, J3 0.1" Header, J4 JST B6B-PH-K-S, J5 JST B6B-PH-K-S, J6 XLR5, M1 Conn_01x04_Male, M2 Conn_01x04_Male, SW1 Power Switch, U1 Pico, U4 TLC59108xPW

Commit message: Update to V2 of Backpack
Parts:
- removed F1: Fuse, Fuse:Fuse_1206_3216Metric_Pad1.42x1.75mm_HandSolder, symbol Device:Fuse
- removed J2: Pololu D36V28F5, MyloLibrary:Pololu D36V28Fx, symbol New_Library:Pololu D36V28F5
- removed SW1: Power Switch, Connector_JST:JST_PH_B2B-PH-K_1x02_P2.00mm_Vertical, symbol Switch:SW_SPST
- added BT2: CR2032, Battery:BatteryHolder_Keystone_1060_1x2032, symbol Device:Battery_Cell
- added C2, C3: 100 nF, Capacitor_SMD:C_0603_1608Metric_Pad1.08x0.95mm_HandSolder, symbol Device:C_Small
- added R4: 931Ω, Resistor_SMD:R_0402_1005Metric_Pad0.72x0.64mm_HandSolder, symbol Device:R_Small_US
- added SW1, SW2: SKRKAHE020, Button_Switch_SMD:SW_Push_SPST_NO_Alps_SKRK, symbol Switch:SW_Push
- added U2: DS3231MZ, Package_SO:SOIC-8_3.9x4.9mm_P1.27mm, symbol Timer_RTC:DS3231MZ
- added U5, U6: TMC2209_SILENTSTEPSTICK, TMC2209 SilentStepStick:MODULE_TMC2209_SILENTSTEPSTICK, symbol TMC2209_SILENTSTEPSTICK:TMC2209_SILENTSTEPSTICK
- BT1: value 10S Li-ion -> 3S Li-ion; footprint Connector_AMASS:AMASS_XT60-M_1x02_P7.20mm_Vertical -> Connector_JST:JST_XH_B2B-XH-AM_1x02_P2.50mm_Vertical
- C1: footprint Capacitor_SMD:C_0805_2012Metric_Pad1.18x1.45mm_HandSolder -> Capacitor_SMD:C_0603_1608Metric_Pad1.08x0.95mm_HandSolder
- D1: value ? -> SD103AWS; footprint Diode_SMD:D_1206_3216Metric -> Diode_SMD:D_SOD-323_HandSoldering
- H1, H2, H3, H4: footprint MountingHole:MountingHole_3.2mm_M3_Pad_Via -> MountingHole:MountingHole_3.2mm_M3_ISO7380; symbol Mechanical:MountingHole_Pad -> Mechanical:MountingHole; now left out of the parts list
- J1: value Pololu D24V10F3 -> Pololu D24V5F3; footprint MyloLibrary:Pololu D24V10Fx -> TMC2209 SilentStepStick:Pololu_D24V5Fx; symbol New_Library:Pololu D24V10F3 -> TMC2209_SILENTSTEPSTICK:Pololu_D24V5Fx
- R1: footprint Resistor_SMD:R_0805_2012Metric -> Resistor_SMD:R_0805_2012Metric_Pad1.20x1.40mm_HandSolder
- R2: value 11k -> 100k; footprint Resistor_SMD:R_0805_2012Metric -> Resistor_SMD:R_0603_1608Metric_Pad0.98x0.95mm_HandSolder
- R3: value 820 -> 30.1k; footprint Resistor_SMD:R_0805_2012Metric -> Resistor_SMD:R_0603_1608Metric_Pad0.98x0.95mm_HandSolder
- U4: value TLC59108xPW -> TLC59108FIPWR
Connections:
- net +12V is gone; now on net +BATT: J4.1 (Pin_1)
- net BUTTON_0 is gone; now on net BUTTON_1: J5.6 (Pin_6), U1.4 (GPIO2)
- net +3V3: now also D1.2 (A), J1.4 (VOUT), C2.1, U2.6 (VBAT), U5.2 (VIO), U6.15 (MS1), U6.2 (VIO); no longer U1.36 (3V3)
- net +BATT: now also BT1.1 (+), J1.2 (VIN), J6.1 (P1), U5.8 (VM), U6.8 (VM); no longer J1.3 (VIN), J6.3 (P3)
- net BAT_VOLTAGE: now also U1.34 (GPIO28_ADC2); no longer U1.31 (GPIO26_ADC0)
- net BR_DIR: now also U1.26 (GPIO20), U6.9 (DIR); no longer U1.16 (GPIO12)
- net BR_STEP: now also U1.27 (GPIO21), U6.10 (STEP); no longer U1.17 (GPIO13)
- net BUTTON_1: no longer J5.5 (Pin_5), U1.5 (GPIO3)
- net BUTTON_2: now also J5.5 (Pin_5), U1.5 (GPIO3); no longer J5.4 (Pin_4), U1.6 (GPIO4)
- net BUTTON_3: now also J5.4 (Pin_4), U1.6 (GPIO4); no longer J5.3 (Pin_3), U1.7 (GPIO5)
- net BUTTON_4: now also J5.3 (Pin_3), U1.7 (GPIO5); no longer J5.2 (Pin_2), U1.9 (GPIO6)
- net GND: now also J1.3 (GND), BT2.2 (-), C2.2, C3.2, R4.1, SW1.1, SW2.1, U2.5 (GND), U5.1 (GND), U5.14 (MS2), U5.15 (MS1), U5.7 (GND), U6.1 (GND), U6.14 (MS2), U6.7 (GND); no longer H1.1, H2.1, H3.1, H4.1, J1.4 (GND), U1.32 (GPIO27_ADC1)
- net M1A+: now also M1.3 (Pin_3), U5.4 (M1A); no longer M1.2 (Pin_2)
- net M1A-: now also M1.4 (Pin_4), U5.3 (M1B); no longer M1.1 (Pin_1)
- net M1B+: now also M1.2 (Pin_2), U5.5 (M2A); no longer M1.3 (Pin_3)
- net M1B-: now also M1.1 (Pin_1), U5.6 (M2B); no longer M1.4 (Pin_4)
- net M2A+: now also M2.3 (Pin_3), U6.4 (M1A); no longer M2.2 (Pin_2)
- net M2A-: now also M2.4 (Pin_4), U6.3 (M1B); no longer M2.1 (Pin_1)
- net M2B+: now also M2.2 (Pin_2), U6.5 (M2A); no longer M2.3 (Pin_3)
- net M2B-: now also M2.1 (Pin_1), U6.6 (M2B); no longer M2.4 (Pin_4)
- net OUT_RX: now also J6.3 (P3), U1.17 (GPIO13); no longer J3.3 (Pin_3), J6.5 (P5), U1.1 (GPIO0)
- net OUT_TX: now also J6.5 (P5), U1.16 (GPIO12); no longer J3.1 (Pin_1), J6.1 (P1), U1.2 (GPIO1)
- net REEL_~{EN}: now also U1.32 (GPIO27_ADC1), U5.16 (~{EN}), U6.16 (~{EN}); no longer U1.21 (GPIO16)
- net S_UART: now also U1.11 (GPIO8), U5.12 (UART), U6.12 (UART); no longer U1.27 (GPIO21)
- net TR_DIR: now also U1.24 (GPIO18), U5.9 (DIR); no longer U1.19 (GPIO14)
- net TR_STEP: now also U1.25 (GPIO19), U5.10 (STEP); no longer U1.20 (GPIO15)
- net at U4.1 (REXT): now also R4.2
- net LED3: now reaches J4.5 (Pin_5), U4.10 (~{OUT3})
- net LED4: now reaches U4.11 (~{OUT4})
- net LED4: now also J4.2 (Pin_2); no longer J4.3 (Pin_3)
- net LED5: now reaches U4.12 (~{OUT5})
- net LED5: now also J4.3 (Pin_3); no longer J4.2 (Pin_2)
- net LED1: now reaches J4.6 (Pin_6), U4.7 (~{OUT1})
- net LED2: now reaches J4.4 (Pin_4), U4.9 (~{OUT2})
- net S_TX: now reaches R1.2
- net S_TX: now also U1.12 (GPIO9); no longer U1.26 (GPIO20)
- net 32KHz: now reaches U1.29 (GPIO22)
- net 32KHz: now also U2.1 (32KHZ)
- net RUN: now reaches U1.30 (RUN)
- net RUN: now also SW1.2
- removed net +5V: D1.2 (A), J1.5 (VOUT)
- net LED_SCL renamed SCL
- net SCL: now also U4.18 (SCL), U2.8 (SCL); no longer U4.19 (SDA)
- net LED_SDA renamed SDA
- net SDA: now also U4.19 (SDA), U2.7 (SDA); no longer U4.18 (SCL)
- new net: BT2.1 (+), C3.1, U2.2 (VCC)
- new net BR_DIAG: U1.19 (GPIO14), U6.18 (DIAG)
- new net BUTTON_5: J5.2 (Pin_2), U1.9 (GPIO6)
- new net DBG_RX: J3.1 (Pin_1), U1.2 (GPIO1)
- new net DBG_TX: J3.3 (Pin_3), U1.1 (GPIO0)
- new net SPRD: U1.31 (GPIO26_ADC0), U5.13 (SPRD), U6.13 (SPRD)
- new net TR_DIAG: U1.20 (GPIO15), U5.18 (DIAG)
- new net ~{RST}: SW2.2, U2.4 (~{RST})
- no-connect marks 19 -> 14
Other:
- removed sheet Stepper Drivers
- note added: "Battery is fused and switched before it arrives on the PCB"
- note added: "Bottom Reel"
- note added: "Top Reel"
- note removed: "Motor 1 Driver"
- note removed: "Motor 2 Driver"
- moved on the sheet: BT1, D1, J4, R2, R3, U1
