File: ProtoPico/mcu.kicad_sch (KiCad schematic)
At the start: 26 parts, among them J3 SM04B-SRSS-TB, SW1 TL3305AF160QG, SW2 TL3305AF160QG, U2 W25Q64JVSSIQ, U3 RP2040, Y1 12MHz 3225 SMD

Commit message: Update to V2 of Backpack
Parts:
- removed R1: 10k, Resistor_SMD:R_0805_2012Metric, symbol Device:R_US
- removed TP1, TP2: TestPoint, TestPoint:TestPoint_Pad_D2.0mm, symbol Connector:TestPoint
- added D17: BAT201M3 RRG, Diode_SMD:D_SOD-323_HandSoldering, symbol Device:D_Schottky
- added J8: JST-SH, Connector_JST:JST_SH_SM03B-SRSS-TB_1x03-1MP_P1.00mm_Horizontal, symbol Connector_Generic_MountingPin:Conn_01x03_MountingPin
- added J9: GPIO, Connector_JST:JST_GH_SM06B-GHS-TB_1x06-1MP_P1.25mm_Horizontal, symbol Connector_Generic_MountingPin:Conn_01x06_MountingPin
- added JP1: Voltage Select, Jumper:SolderJumper-3_P1.3mm_Open_RoundedPad1.0x1.5mm, symbol Jumper:SolderJumper_3_Open
- added R16, R17: 100, Resistor_SMD:R_0402_1005Metric, symbol Device:R_Small_US
- C13, C14: footprint Capacitor_SMD:C_0805_2012Metric -> Capacitor_SMD:C_0402_1005Metric
- J7: renamed from J3; footprint ProtoPico_Footprints:JST_SH_SM04B-SRSS-TB_1x04-1MP_P1.00mm_Horizontal -> Connector_JST:JST_PH_S4B-PH-SM4-TB_1x04-1MP_P2.00mm_Horizontal
- R7: renamed from R3; footprint Resistor_SMD:R_0805_2012Metric -> Resistor_SMD:R_0402_1005Metric
- renumbered C6 to C10, C9 to C11, C3 to C12, C12 to C2, C4 to C3, C2 to C4, C11 to C5, C5 to C6, C10 to C7, C7 to C9, R2 to R4, R4 to R5, R5 to R6
Connections:
- net UART0 RX is gone; now on net Fan_Tach: U3.16 (GPIO13)
- net UART0 TX is gone; now on net Fan_PWM: U3.15 (GPIO12)
- net +3.3V: now also JP1.1 (A)
- net +5V: now also JP1.3 (B); no longer J7.1 (Pin_1)
- net Fan_PWM: no longer U3.18 (GPIO15)
- net Fan_Tach: no longer U3.17 (GPIO14)
- net GND: now also J8.2 (Pin_2), J8.MP (MountPin), J9.1 (Pin_1), J9.MP (MountPin)
- net SWCLK: now also R16.2
- net SWD: now also R17.2
- net GPIO10: now reaches U3.13 (GPIO10)
- net GPIO10: now also J9.5 (Pin_5)
- net GPIO11: now reaches U3.14 (GPIO11)
- net GPIO11: now also J9.6 (Pin_6)
- net UART1 RX renamed GPIO9
- net GPIO9: now also J9.4 (Pin_4)
- net UART1 TX renamed GPIO8
- net GPIO8: now also J9.3 (Pin_3)
- new net: J8.1 (Pin_1), R16.1
- new net: J8.3 (Pin_3), R17.1
- new net: J9.2 (Pin_2), JP1.2 (C)
- new net +BATT: D17.1 (K)
- new net 5V_EN: U3.17 (GPIO14)
- new net 5V_PG: U3.18 (GPIO15)
- new net VUSB: D17.2 (A), J7.1 (Pin_1)
- no-connect marks 17 -> 15
Other:
- moved on the sheet: J7, R4, SW1
